File: hardware/pcba-rev-a/elec/layout/default/default.kicad_pcb (KiCad board)
At the start: 2 copper layers, 20 parts

Commit message: Rev A: real parts bound — 172 components, 29 LCSC BOM lines, build green
15 parts created from LCSC via ato create part: Omron G6K-2F-Y-TR DC5
(C47190) x64, PAN CHANG SIP-1A05 reed (C10496) x27, TPIC6B595DWR x12,
TPS54331/62086/7A4901 regulators + support passives (inductors, boot
cap, feedback dividers), TPS3823 watchdog, 24AA025UID EEPROM, INA219
telemetry, TLV3502 comparators x8, BAV99 steering x8, SMAJ24CA x8,
SMBJ33A, 0805L010YR PTC x8. Pinouts datasheet-verified (G6K terminal
arrangement read from the Omron datasheet render; multiple original
guesses corrected). Constraint solver picked 0.1% thin-film cal
references. Lesson: atomic parts must not be subclassed (footprint
path resolution) - pin aliases live in the part files.

Remaining unbound (documented): 24V fuse, Pico + SEAF local parts,
J-connectors. Substitution notes: unshielded reeds, 100mA PTC.

Co-Authored-By: Claude Fable 5 <noreply@anthropic.com>
Parts:
- added C1: 100nF ±10%, YAGEO_CC0603KRX7R9BB104:C0603, F.Cu at (1340.0, -10.0)
- added C2: 10nF ±10%, FH_0603B103K500NT:C0603, F.Cu at (1340.0, -20.0)
- added D1: , Littelfuse_SMBJ33A:SMB_L4.6-W3.6-LS5.3-RD, F.Cu at (0.00, 0.00)
- added D10: , Nexperia_BAV99_215:SOT-23-3_L2.9-W1.6-P1.90-LS2.8-BR, F.Cu at (1100.0, 0.00)
- added D11: , Littelfuse_SMAJ24CA:SMA_L4.4-W2.6-LS5.0-BI, F.Cu at (1110.0, 0.00)
- added D12: , Nexperia_BAV99_215:SOT-23-3_L2.9-W1.6-P1.90-LS2.8-BR, F.Cu at (1130.0, 0.00)
- added D13: , Littelfuse_SMAJ24CA:SMA_L4.4-W2.6-LS5.0-BI, F.Cu at (1140.0, 0.00)
- added D14: , Nexperia_BAV99_215:SOT-23-3_L2.9-W1.6-P1.90-LS2.8-BR, F.Cu at (1160.0, 0.00)
- added D15: , Littelfuse_SMAJ24CA:SMA_L4.4-W2.6-LS5.0-BI, F.Cu at (1170.0, 0.00)
- added D16: , Nexperia_BAV99_215:SOT-23-3_L2.9-W1.6-P1.90-LS2.8-BR, F.Cu at (1190.0, 0.00)
- added D17: , Littelfuse_SMAJ24CA:SMA_L4.4-W2.6-LS5.0-BI, F.Cu at (1200.0, 0.00)
- added D2: , Nexperia_BAV99_215:SOT-23-3_L2.9-W1.6-P1.90-LS2.8-BR, F.Cu at (1250.0, 0.00)
- added D3: , Littelfuse_SMAJ24CA:SMA_L4.4-W2.6-LS5.0-BI, F.Cu at (1260.0, 0.00)
- added D4: , Nexperia_BAV99_215:SOT-23-3_L2.9-W1.6-P1.90-LS2.8-BR, F.Cu at (1220.0, 0.00)
- added D5: , Littelfuse_SMAJ24CA:SMA_L4.4-W2.6-LS5.0-BI, F.Cu at (1230.0, 0.00)
- added D6: , Nexperia_BAV99_215:SOT-23-3_L2.9-W1.6-P1.90-LS2.8-BR, F.Cu at (1310.0, 0.00)
- added D7: , Littelfuse_SMAJ24CA:SMA_L4.4-W2.6-LS5.0-BI, F.Cu at (1320.0, 0.00)
- added D8: , Nexperia_BAV99_215:SOT-23-3_L2.9-W1.6-P1.90-LS2.8-BR, F.Cu at (1280.0, 0.00)
- added D9: , Littelfuse_SMAJ24CA:SMA_L4.4-W2.6-LS5.0-BI, F.Cu at (1290.0, 0.00)
- added K1: , Omron_Electronics_G6K_2F_Y_TR_DC5:RELAY-SMD_G6K-2F-X-XX, F.Cu at (740.0, 0.00)
- added K10: , Omron_Electronics_G6K_2F_Y_TR_DC5:RELAY-SMD_G6K-2F-X-XX, F.Cu at (750.0, 0.00)
- added K11: , Omron_Electronics_G6K_2F_Y_TR_DC5:RELAY-SMD_G6K-2F-X-XX, F.Cu at (760.0, 0.00)
- added K12: , Omron_Electronics_G6K_2F_Y_TR_DC5:RELAY-SMD_G6K-2F-X-XX, F.Cu at (630.0, 0.00)
- added K13: , Omron_Electronics_G6K_2F_Y_TR_DC5:RELAY-SMD_G6K-2F-X-XX, F.Cu at (660.0, 0.00)
- added K14: , Omron_Electronics_G6K_2F_Y_TR_DC5:RELAY-SMD_G6K-2F-X-XX, F.Cu at (670.0, 0.00)
- added K15: , PAN_CHANG_SIP_1A05:RELAY-TH_SIP-1A05, F.Cu at (710.0, 0.00)
- added K16: , PAN_CHANG_SIP_1A05:RELAY-TH_SIP-1A05, F.Cu at (720.0, 0.00)
- added K17: , PAN_CHANG_SIP_1A05:RELAY-TH_SIP-1A05, F.Cu at (730.0, 0.00)
- added K18: , Omron_Electronics_G6K_2F_Y_TR_DC5:RELAY-SMD_G6K-2F-X-XX, F.Cu at (680.0, 0.00)
- added K19: , Omron_Electronics_G6K_2F_Y_TR_DC5:RELAY-SMD_G6K-2F-X-XX, F.Cu at (690.0, 0.00)
- added K2: , Omron_Electronics_G6K_2F_Y_TR_DC5:RELAY-SMD_G6K-2F-X-XX, F.Cu at (770.0, 0.00)
- added K20: , Omron_Electronics_G6K_2F_Y_TR_DC5:RELAY-SMD_G6K-2F-X-XX, F.Cu at (700.0, 0.00)
- added K21: , Omron_Electronics_G6K_2F_Y_TR_DC5:RELAY-SMD_G6K-2F-X-XX, F.Cu at (640.0, 0.00)
- added K22: , Omron_Electronics_G6K_2F_Y_TR_DC5:RELAY-SMD_G6K-2F-X-XX, F.Cu at (650.0, 0.00)
- added K23: , Omron_Electronics_G6K_2F_Y_TR_DC5:RELAY-SMD_G6K-2F-X-XX, F.Cu at (960.0, 0.00)
- added K24: , Omron_Electronics_G6K_2F_Y_TR_DC5:RELAY-SMD_G6K-2F-X-XX, F.Cu at (990.0, 0.00)
- added K25: , Omron_Electronics_G6K_2F_Y_TR_DC5:RELAY-SMD_G6K-2F-X-XX, F.Cu at (1000.0, 0.00)
- added K26: , PAN_CHANG_SIP_1A05:RELAY-TH_SIP-1A05, F.Cu at (1040.0, 0.00)
- added K27: , PAN_CHANG_SIP_1A05:RELAY-TH_SIP-1A05, F.Cu at (1050.0, 0.00)
- added K28: , PAN_CHANG_SIP_1A05:RELAY-TH_SIP-1A05, F.Cu at (1060.0, 0.00)
- added K29: , Omron_Electronics_G6K_2F_Y_TR_DC5:RELAY-SMD_G6K-2F-X-XX, F.Cu at (1010.0, 0.00)
- added K3: , Omron_Electronics_G6K_2F_Y_TR_DC5:RELAY-SMD_G6K-2F-X-XX, F.Cu at (780.0, 0.00)
- added K30: , Omron_Electronics_G6K_2F_Y_TR_DC5:RELAY-SMD_G6K-2F-X-XX, F.Cu at (1020.0, 0.00)
- added K31: , Omron_Electronics_G6K_2F_Y_TR_DC5:RELAY-SMD_G6K-2F-X-XX, F.Cu at (1030.0, 0.00)
- added K32: , Omron_Electronics_G6K_2F_Y_TR_DC5:RELAY-SMD_G6K-2F-X-XX, F.Cu at (970.0, 0.00)
- added K33: , Omron_Electronics_G6K_2F_Y_TR_DC5:RELAY-SMD_G6K-2F-X-XX, F.Cu at (980.0, 0.00)
- added K34: , Omron_Electronics_G6K_2F_Y_TR_DC5:RELAY-SMD_G6K-2F-X-XX, F.Cu at (850.0, 0.00)
- added K35: , Omron_Electronics_G6K_2F_Y_TR_DC5:RELAY-SMD_G6K-2F-X-XX, F.Cu at (880.0, 0.00)
- added K36: , Omron_Electronics_G6K_2F_Y_TR_DC5:RELAY-SMD_G6K-2F-X-XX, F.Cu at (890.0, 0.00)
- added K37: , PAN_CHANG_SIP_1A05:RELAY-TH_SIP-1A05, F.Cu at (930.0, 0.00)
- added K38: , PAN_CHANG_SIP_1A05:RELAY-TH_SIP-1A05, F.Cu at (940.0, 0.00)
- added K39: , PAN_CHANG_SIP_1A05:RELAY-TH_SIP-1A05, F.Cu at (950.0, 0.00)
- added K4: , PAN_CHANG_SIP_1A05:RELAY-TH_SIP-1A05, F.Cu at (820.0, 0.00)
- added K40: , Omron_Electronics_G6K_2F_Y_TR_DC5:RELAY-SMD_G6K-2F-X-XX, F.Cu at (900.0, 0.00)
- added K41: , Omron_Electronics_G6K_2F_Y_TR_DC5:RELAY-SMD_G6K-2F-X-XX, F.Cu at (910.0, 0.00)
- added K42: , Omron_Electronics_G6K_2F_Y_TR_DC5:RELAY-SMD_G6K-2F-X-XX, F.Cu at (920.0, 0.00)
- added K43: , Omron_Electronics_G6K_2F_Y_TR_DC5:RELAY-SMD_G6K-2F-X-XX, F.Cu at (860.0, 0.00)
- added K44: , Omron_Electronics_G6K_2F_Y_TR_DC5:RELAY-SMD_G6K-2F-X-XX, F.Cu at (870.0, 0.00)
- added K45: , Omron_Electronics_G6K_2F_Y_TR_DC5:RELAY-SMD_G6K-2F-X-XX, F.Cu at (190.0, 0.00)
- added K46: , Omron_Electronics_G6K_2F_Y_TR_DC5:RELAY-SMD_G6K-2F-X-XX, F.Cu at (220.0, 0.00)
- added K47: , Omron_Electronics_G6K_2F_Y_TR_DC5:RELAY-SMD_G6K-2F-X-XX, F.Cu at (230.0, 0.00)
- added K48: , PAN_CHANG_SIP_1A05:RELAY-TH_SIP-1A05, F.Cu at (270.0, 0.00)
- added K49: , PAN_CHANG_SIP_1A05:RELAY-TH_SIP-1A05, F.Cu at (280.0, 0.00)
- added K5: , PAN_CHANG_SIP_1A05:RELAY-TH_SIP-1A05, F.Cu at (830.0, 0.00)
- added K50: , PAN_CHANG_SIP_1A05:RELAY-TH_SIP-1A05, F.Cu at (290.0, 0.00)
- added K51: , Omron_Electronics_G6K_2F_Y_TR_DC5:RELAY-SMD_G6K-2F-X-XX, F.Cu at (240.0, 0.00)
- added K52: , Omron_Electronics_G6K_2F_Y_TR_DC5:RELAY-SMD_G6K-2F-X-XX, F.Cu at (250.0, 0.00)
- added K53: , Omron_Electronics_G6K_2F_Y_TR_DC5:RELAY-SMD_G6K-2F-X-XX, F.Cu at (260.0, 0.00)
- added K54: , Omron_Electronics_G6K_2F_Y_TR_DC5:RELAY-SMD_G6K-2F-X-XX, F.Cu at (200.0, 0.00)
- added K55: , Omron_Electronics_G6K_2F_Y_TR_DC5:RELAY-SMD_G6K-2F-X-XX, F.Cu at (210.0, 0.00)
- added K56: , Omron_Electronics_G6K_2F_Y_TR_DC5:RELAY-SMD_G6K-2F-X-XX, F.Cu at (300.0, 0.00)
- added K57: , Omron_Electronics_G6K_2F_Y_TR_DC5:RELAY-SMD_G6K-2F-X-XX, F.Cu at (330.0, 0.00)
- added K58: , Omron_Electronics_G6K_2F_Y_TR_DC5:RELAY-SMD_G6K-2F-X-XX, F.Cu at (340.0, 0.00)
- added K59: , PAN_CHANG_SIP_1A05:RELAY-TH_SIP-1A05, F.Cu at (380.0, 0.00)
- added K6: , PAN_CHANG_SIP_1A05:RELAY-TH_SIP-1A05, F.Cu at (840.0, 0.00)
- added K60: , PAN_CHANG_SIP_1A05:RELAY-TH_SIP-1A05, F.Cu at (390.0, 0.00)
- added K61: , PAN_CHANG_SIP_1A05:RELAY-TH_SIP-1A05, F.Cu at (400.0, 0.00)
- added K62: , Omron_Electronics_G6K_2F_Y_TR_DC5:RELAY-SMD_G6K-2F-X-XX, F.Cu at (350.0, 0.00)
- added K63: , Omron_Electronics_G6K_2F_Y_TR_DC5:RELAY-SMD_G6K-2F-X-XX, F.Cu at (360.0, 0.00)
- added K64: , Omron_Electronics_G6K_2F_Y_TR_DC5:RELAY-SMD_G6K-2F-X-XX, F.Cu at (370.0, 0.00)
- added K65: , Omron_Electronics_G6K_2F_Y_TR_DC5:RELAY-SMD_G6K-2F-X-XX, F.Cu at (310.0, 0.00)
- added K66: , Omron_Electronics_G6K_2F_Y_TR_DC5:RELAY-SMD_G6K-2F-X-XX, F.Cu at (320.0, 0.00)
- added K67: , Omron_Electronics_G6K_2F_Y_TR_DC5:RELAY-SMD_G6K-2F-X-XX, F.Cu at (410.0, 0.00)
- added K68: , Omron_Electronics_G6K_2F_Y_TR_DC5:RELAY-SMD_G6K-2F-X-XX, F.Cu at (440.0, 0.00)
- added K69: , Omron_Electronics_G6K_2F_Y_TR_DC5:RELAY-SMD_G6K-2F-X-XX, F.Cu at (450.0, 0.00)
- added K7: , Omron_Electronics_G6K_2F_Y_TR_DC5:RELAY-SMD_G6K-2F-X-XX, F.Cu at (790.0, 0.00)
- added K70: , PAN_CHANG_SIP_1A05:RELAY-TH_SIP-1A05, F.Cu at (490.0, 0.00)
- added K71: , PAN_CHANG_SIP_1A05:RELAY-TH_SIP-1A05, F.Cu at (500.0, 0.00)
- added K72: , PAN_CHANG_SIP_1A05:RELAY-TH_SIP-1A05, F.Cu at (510.0, 0.00)
- added K73: , Omron_Electronics_G6K_2F_Y_TR_DC5:RELAY-SMD_G6K-2F-X-XX, F.Cu at (460.0, 0.00)
- added K74: , Omron_Electronics_G6K_2F_Y_TR_DC5:RELAY-SMD_G6K-2F-X-XX, F.Cu at (470.0, 0.00)
- added K75: , Omron_Electronics_G6K_2F_Y_TR_DC5:RELAY-SMD_G6K-2F-X-XX, F.Cu at (480.0, 0.00)
- added K76: , Omron_Electronics_G6K_2F_Y_TR_DC5:RELAY-SMD_G6K-2F-X-XX, F.Cu at (420.0, 0.00)
- added K77: , Omron_Electronics_G6K_2F_Y_TR_DC5:RELAY-SMD_G6K-2F-X-XX, F.Cu at (430.0, 0.00)
- added K78: , Omron_Electronics_G6K_2F_Y_TR_DC5:RELAY-SMD_G6K-2F-X-XX, F.Cu at (520.0, 0.00)
- added K79: , Omron_Electronics_G6K_2F_Y_TR_DC5:RELAY-SMD_G6K-2F-X-XX, F.Cu at (550.0, 0.00)
- added K8: , Omron_Electronics_G6K_2F_Y_TR_DC5:RELAY-SMD_G6K-2F-X-XX, F.Cu at (800.0, 0.00)
- added K80: , Omron_Electronics_G6K_2F_Y_TR_DC5:RELAY-SMD_G6K-2F-X-XX, F.Cu at (560.0, 0.00)
- added K81: , PAN_CHANG_SIP_1A05:RELAY-TH_SIP-1A05, F.Cu at (600.0, 0.00)
- added K82: , PAN_CHANG_SIP_1A05:RELAY-TH_SIP-1A05, F.Cu at (610.0, 0.00)
- added K83: , PAN_CHANG_SIP_1A05:RELAY-TH_SIP-1A05, F.Cu at (620.0, 0.00)
- added K84: , Omron_Electronics_G6K_2F_Y_TR_DC5:RELAY-SMD_G6K-2F-X-XX, F.Cu at (570.0, 0.00)
- added K85: , Omron_Electronics_G6K_2F_Y_TR_DC5:RELAY-SMD_G6K-2F-X-XX, F.Cu at (580.0, 0.00)
- added K86: , Omron_Electronics_G6K_2F_Y_TR_DC5:RELAY-SMD_G6K-2F-X-XX, F.Cu at (590.0, 0.00)
- added K87: , Omron_Electronics_G6K_2F_Y_TR_DC5:RELAY-SMD_G6K-2F-X-XX, F.Cu at (530.0, 0.00)
- added K88: , Omron_Electronics_G6K_2F_Y_TR_DC5:RELAY-SMD_G6K-2F-X-XX, F.Cu at (540.0, 0.00)
- added K89: , PAN_CHANG_SIP_1A05:RELAY-TH_SIP-1A05, F.Cu at (1070.0, 0.00)
- added K9: , Omron_Electronics_G6K_2F_Y_TR_DC5:RELAY-SMD_G6K-2F-X-XX, F.Cu at (810.0, 0.00)
- added K90: , PAN_CHANG_SIP_1A05:RELAY-TH_SIP-1A05, F.Cu at (1080.0, 0.00)
- added K91: , PAN_CHANG_SIP_1A05:RELAY-TH_SIP-1A05, F.Cu at (1090.0, 0.00)
- added L1: L 2.2µH ±20%, cjiang_FTC252012S2R2MBCA:IND-SMD_L2.5-W2.0_MHCHL2520, F.Cu at (1340.0, -100.0)
- added L2: L 10µH ±20%, Murata_Electronics_LQM18FN100M00D:L0603, F.Cu at (1340.0, -90.0)
- added R21: 100kΩ ±1%, UNI_ROYAL_0402WGF1003TCE:R0402, F.Cu at (1340.0, -240.0)
- added R22: 1MΩ ±1%, UNI_ROYAL_0603WAF1004T5E:R0603, F.Cu at (1340.0, -250.0)
- added R23: 100kΩ ±1%, UNI_ROYAL_0402WGF1003TCE:R0402, F.Cu at (1340.0, -260.0)
- added R24: 1MΩ ±1%, UNI_ROYAL_0603WAF1004T5E:R0603, F.Cu at (1340.0, -270.0)
- added R25: 1kΩ ±0.1%, YAGEO_RT0603BRD071KL:R0603, F.Cu at (1340.0, -290.0)
- added R26: 100kΩ ±0.1%, Viking_Tech_ARG03BTC1003:R0603, F.Cu at (1340.0, -280.0)
- added U1: , Microchip_Tech_24AA025UIDT_I_OT:SOT-23-6_L2.9-W1.6-P0.95-LS2.8-BR, F.Cu at (60.0, 0.00)
- added U10: , Texas_Instruments_TPIC6B595DWR:SOIC-20_L13.0-W7.6-P1.27-LS10.3-BL, F.Cu at (150.0, 0.00)
- added U11: , Texas_Instruments_TPIC6B595DWR:SOIC-20_L13.0-W7.6-P1.27-LS10.3-BL, F.Cu at (160.0, 0.00)
- added U12: , Texas_Instruments_TPIC6B595DWR:SOIC-20_L13.0-W7.6-P1.27-LS10.3-BL, F.Cu at (170.0, 0.00)
- added U13: , Texas_Instruments_TPIC6B595DWR:SOIC-20_L13.0-W7.6-P1.27-LS10.3-BL, F.Cu at (180.0, 0.00)
- added U14: , Texas_Instruments_TPS3823_33DBVR:SOT-23-5_L3.0-W1.7-P0.95-LS2.8-BL, F.Cu at (50.0, 0.00)
- added U15: , Texas_Instruments_TPS62086RLTR:VSON-7_L2.0-W2.0-P0.5-TL, F.Cu at (20.0, 0.00)
- added U16: , Texas_Instruments_TPS54331DR:SOIC-8_L5.0-W4.0-P1.27-LS6.0-BL, F.Cu at (10.0, 0.00)
- added U17: , Texas_Instruments_INA219AIDCNR:SOT-23-8_L3.0-W1.7-P0.65-LS2.8-BR, F.Cu at (40.0, 0.00)
- added U18: , Texas_Instruments_TPS7A4901DGNR:HVSSOP-8_L3.0-W3.0-P0.65-LS4.9-BL-EP_DGN0008D, F.Cu at (30.0, 0.00)
- added U19: , Texas_Instruments_TLV3502AIDR:SOIC-8_L4.9-W3.9-P1.27-LS6.0-BL, F.Cu at (1270.0, 0.00)
- added U2: , Texas_Instruments_TPIC6B595DWR:SOIC-20_L13.0-W7.6-P1.27-LS10.3-BL, F.Cu at (70.0, 0.00)
- added U20: , Texas_Instruments_TLV3502AIDR:SOIC-8_L4.9-W3.9-P1.27-LS6.0-BL, F.Cu at (1240.0, 0.00)
- added U21: , Texas_Instruments_TLV3502AIDR:SOIC-8_L4.9-W3.9-P1.27-LS6.0-BL, F.Cu at (1330.0, 0.00)
- added U22: , Texas_Instruments_TLV3502AIDR:SOIC-8_L4.9-W3.9-P1.27-LS6.0-BL, F.Cu at (1300.0, 0.00)
- added U23: , Texas_Instruments_TLV3502AIDR:SOIC-8_L4.9-W3.9-P1.27-LS6.0-BL, F.Cu at (1120.0, 0.00)
- added U24: , Texas_Instruments_TLV3502AIDR:SOIC-8_L4.9-W3.9-P1.27-LS6.0-BL, F.Cu at (1150.0, 0.00)
- added U25: , Texas_Instruments_TLV3502AIDR:SOIC-8_L4.9-W3.9-P1.27-LS6.0-BL, F.Cu at (1180.0, 0.00)
- added U26: , Texas_Instruments_TLV3502AIDR:SOIC-8_L4.9-W3.9-P1.27-LS6.0-BL, F.Cu at (1210.0, 0.00)
- added U27: , Littelfuse_0805L010YR:F0805, F.Cu at (50.0, 0.00)
- added U28: , Littelfuse_0805L010YR:F0805, F.Cu at (40.0, 0.00)
- added U29: , Littelfuse_0805L010YR:F0805, F.Cu at (70.0, 0.00)
- added U3: , Texas_Instruments_TPIC6B595DWR:SOIC-20_L13.0-W7.6-P1.27-LS10.3-BL, F.Cu at (80.0, 0.00)
- added U30: , Littelfuse_0805L010YR:F0805, F.Cu at (60.0, 0.00)
- added U31: , Littelfuse_0805L010YR:F0805, F.Cu at (0.00, 0.00)
- added U32: , Littelfuse_0805L010YR:F0805, F.Cu at (10.0, 0.00)
- added U33: , Littelfuse_0805L010YR:F0805, F.Cu at (20.0, 0.00)
- added U34: , Littelfuse_0805L010YR:F0805, F.Cu at (30.0, 0.00)
- added U4: , Texas_Instruments_TPIC6B595DWR:SOIC-20_L13.0-W7.6-P1.27-LS10.3-BL, F.Cu at (90.0, 0.00)
- added U5: , Texas_Instruments_TPIC6B595DWR:SOIC-20_L13.0-W7.6-P1.27-LS10.3-BL, F.Cu at (100.0, 0.00)
- added U6: , Texas_Instruments_TPIC6B595DWR:SOIC-20_L13.0-W7.6-P1.27-LS10.3-BL, F.Cu at (110.0, 0.00)
- added U7: , Texas_Instruments_TPIC6B595DWR:SOIC-20_L13.0-W7.6-P1.27-LS10.3-BL, F.Cu at (120.0, 0.00)
- added U8: , Texas_Instruments_TPIC6B595DWR:SOIC-20_L13.0-W7.6-P1.27-LS10.3-BL, F.Cu at (130.0, 0.00)
- added U9: , Texas_Instruments_TPIC6B595DWR:SOIC-20_L13.0-W7.6-P1.27-LS10.3-BL, F.Cu at (140.0, 0.00)
- R10, R12, R14, R16, R18: footprint UNI_ROYAL_0402WGF1004TCE:R0402 -> UNI_ROYAL_0603WAF1004T5E:R0603
- R19: value 1kΩ ±1% -> 100kΩ ±1%; footprint UNI_ROYAL_0805W8F1001T5E:R0805 -> UNI_ROYAL_0402WGF1003TCE:R0402
- R2: value 50mΩ ±1% -> 15.8kΩ ±1%; footprint UNI_ROYAL_1206W3F500MT5E:R1206 -> FOJAN_FRC0603F1582TS:R0603
- R20: value 100kΩ ±1% -> 1MΩ ±1%; footprint UNI_ROYAL_0805W8F1003T5E:R0805 -> UNI_ROYAL_0603WAF1004T5E:R0603
- R4: value 1MΩ ±1% -> 2kΩ ±1%; footprint UNI_ROYAL_0402WGF1004TCE:R0402 -> UNI_ROYAL_0603WAF2001T5E:R0603
- R5: value 100kΩ ±1% -> 10.5kΩ ±1%; footprint UNI_ROYAL_0402WGF1003TCE:R0402 -> UNI_ROYAL_0402WGF1052TCE:R0402
- R6: value 1MΩ ±1% -> 20.5kΩ ±1%; footprint UNI_ROYAL_0402WGF1004TCE:R0402 -> FOJAN_FRC0603F2052TS:R0603
- R7: value 100kΩ ±1% -> 35.7kΩ ±1%; footprint UNI_ROYAL_0402WGF1003TCE:R0402 -> FOJAN_FRC0603F3572TS:R0603
- R8: value 1MΩ ±1% -> 50mΩ ±1%; footprint UNI_ROYAL_0402WGF1004TCE:R0402 -> UNI_ROYAL_1206W3F500MT5E:R1206
- moved R20 1340.9 mm to (1340.0, -230.0)
- moved R10 1340.6 mm to (1340.0, -130.0)
- moved R11 1340.6 mm to (1340.0, -140.0)
- moved R12 1340.6 mm to (1340.0, -150.0)
- moved R13 1340.6 mm to (1340.0, -160.0)
- moved R14 1340.6 mm to (1340.0, -170.0)
- moved R15 1340.6 mm to (1340.0, -180.0)
- moved R16 1340.6 mm to (1340.0, -190.0)
- moved R17 1340.6 mm to (1340.0, -200.0)
- moved R18 1340.6 mm to (1340.0, -210.0)
- moved R2 1340.6 mm to (1340.0, -50.0)
- moved R3 1340.6 mm to (1340.0, -60.0)
- moved R8 1340.6 mm to (1340.0, -110.0)
- moved R9 1340.6 mm to (1340.0, -120.0)
- moved R19 1340.3 mm to (1340.0, -220.0)
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Connections:
- net prot_ksp-vin renamed IN_Apos
- net prot_p1-vin renamed prot_kfp-IN_Apos
- net prot_p2-vin renamed prot_ksn-IN_Apos
- net prot_p3-vin renamed prot_ksp-IN_Apos
- net prot_p4-vin renamed prot_p1-IN_Apos
- R10 pad 1: node-3 -> node
- R12 pad 1: node-4 -> node-1
- R14 pad 1: node-5 -> node-2
- R16 pad 1: node-6 -> node-3
- R18 pad 1: node-7 -> node-4
- R19 pad 1: refs-no -> prot_p2-IN_Apos
- R2 pad 1: vin -> FB
- R2 pad 2: v5_coil-hv -> lv
- R20 pad 1: no -> node-5
- R20 pad 2: lv -> prot_p2-IN_Apos
- R3 pad 1: prot_kfn-vin -> hv
- R3 pad 2: lv -> FB
- R4 pad 1: node -> VSENSE
- R4 pad 2: prot_kfn-vin -> lv
- R5 pad 1: prot_kfp-vin -> EN
- R5 pad 2: lv -> VSENSE
- R6 pad 1: node-1 -> power-FB
- R6 pad 2: prot_kfp-vin -> lv
- R7 pad 1: prot_ksn-vin -> v3v3-hv
- R7 pad 2: lv -> power-FB
- R8 pad 1: node-2 -> EN
- R8 pad 2: prot_ksn-vin -> sel_p4-coil_bus-hv

Commit message: Rev A: complete netlist — local parts, 91-channel coil map, layout chain
- Local atomic parts (has_part_removed = buyer-furnished): Pico 2 module
  (KiCad official footprint + generated symbol), SEAF14 blind-mate
  (custom footprint), 2/4/8-pin headers for the instrument edge (BNC
  substitution note: bench Rev A uses headers; panel BNCs at DVT).
- Coil control plumbed: 91 relay coil sinks wired to TPIC6B595 drains
  through LaneSelector/Matrix/Control signal exposure; channel map in
  coil-channel-map.md (drains 1-88 = trees p1..ksn x 11 lanes, 89-91 =
  reference block, 92-96 spare) - firmware shares this table.
- Layout chain established: atopile owns elec/layout/default (pristine
  format); placement/zones/routing on derived rev-a-routed.kicad_pcb via
  place_and_zone.py (KiCad 10 writes tokens atopile cannot re-read).
  GND pour In1+B.Cu, coil rail pour In2, outline + mounting holes.
  Freerouting toolchain installed (temurin + freerouting 1.9.0).

Co-Authored-By: Claude Fable 5 <noreply@anthropic.com>
Parts:
- added J1: , Samtec_SEAF14:SEAF14, F.Cu at (200.0, 0.00)
- added J2: , Header_1x02:PinHeader_1x02_P2.54mm_Vertical, F.Cu at (1440.0, 0.00)
- added J3: , Header_1x02:PinHeader_1x02_P2.54mm_Vertical, F.Cu at (1450.0, 0.00)
- added J4: , Header_1x02:PinHeader_1x02_P2.54mm_Vertical, F.Cu at (1460.0, 0.00)
- added J5: , Header_1x04:PinHeader_1x04_P2.54mm_Vertical, F.Cu at (1470.0, 0.00)
- added J6: , Header_1x08:PinHeader_1x08_P2.54mm_Vertical, F.Cu at (1480.0, 0.00)
- added J7: , Header_1x02:PinHeader_1x02_P2.54mm_Vertical, F.Cu at (1490.0, 0.00)
- added U35: , Littelfuse_0805L010YR:F0805, F.Cu at (1240.0, 0.00)
- U14: footprint Texas_Instruments_TPS3823_33DBVR:SOT-23-5_L3.0-W1.7-P0.95-LS2.8-BL -> Texas_Instruments_TPIC6B595DWR:SOIC-20_L13.0-W7.6-P1.27-LS10.3-BL
- U15: footprint Texas_Instruments_TPS62086RLTR:VSON-7_L2.0-W2.0-P0.5-TL -> Texas_Instruments_TPS3823_33DBVR:SOT-23-5_L3.0-W1.7-P0.95-LS2.8-BL
- U16: footprint Texas_Instruments_TPS54331DR:SOIC-8_L5.0-W4.0-P1.27-LS6.0-BL -> Texas_Instruments_TPS62086RLTR:VSON-7_L2.0-W2.0-P0.5-TL
- U17: footprint Texas_Instruments_INA219AIDCNR:SOT-23-8_L3.0-W1.7-P0.65-LS2.8-BR -> Texas_Instruments_TPS54331DR:SOIC-8_L5.0-W4.0-P1.27-LS6.0-BL
- U18: footprint Texas_Instruments_TPS7A4901DGNR:HVSSOP-8_L3.0-W3.0-P0.65-LS4.9-BL-EP_DGN0008D -> Texas_Instruments_INA219AIDCNR:SOT-23-8_L3.0-W1.7-P0.65-LS2.8-BR
- U19: footprint Texas_Instruments_TLV3502AIDR:SOIC-8_L4.9-W3.9-P1.27-LS6.0-BL -> Texas_Instruments_TPS7A4901DGNR:HVSSOP-8_L3.0-W3.0-P0.65-LS4.9-BL-EP_DGN0008D
- U2: footprint Texas_Instruments_TPIC6B595DWR:SOIC-20_L13.0-W7.6-P1.27-LS10.3-BL -> RaspberryPi_Pico2:RaspberryPi_Pico_SMD_HandSolder
- U21, U23, U25: footprint Texas_Instruments_TLV3502AIDR:SOIC-8_L4.9-W3.9-P1.27-LS6.0-BL -> Littelfuse_0805L010YR:F0805
- U28, U30, U32, U34: footprint Littelfuse_0805L010YR:F0805 -> Texas_Instruments_TLV3502AIDR:SOIC-8_L4.9-W3.9-P1.27-LS6.0-BL
- moved U27 1310.0 mm to (1360.0, 0.00)
- moved U19 1240.0 mm to (30.0, 0.00)
- moved U34 1240.0 mm to (1270.0, 0.00)
- moved U32 1220.0 mm to (1230.0, 0.00)
- moved U33 1180.0 mm to (1200.0, 0.00)
- moved U31 1160.0 mm to (1160.0, 0.00)
- moved U30 1130.0 mm to (1190.0, 0.00)
- moved U28 1110.0 mm to (1150.0, 0.00)
- moved U29 1050.0 mm to (1120.0, 0.00)
- moved U24 280.0 mm to (1430.0, 0.00)
- moved U25 220.0 mm to (1400.0, 0.00)
- moved U26 180.0 mm to (1390.0, 0.00)
- moved C1 160.0 mm to (1500.0, -10.0)
- moved C2 160.0 mm to (1500.0, -20.0)
- moved L1 160.0 mm to (1500.0, -100.0)
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Connections:
- K1 pad 8: coil_n -> sink_kfn_bank
- K10 pad 8: matrix.sel_kfn.k_scope_a-coil_n -> sink_kfn_scope_a
- K11 pad 8: matrix.sel_kfn.k_scope_b-coil_n -> sink_kfn_scope_b
- K12 pad 8: matrix.sel_kfp.k_bank-coil_n -> sink_kfp_bank
- K13 pad 8: matrix.sel_kfp.k_daq_1-coil_n -> coil_n-13
- K14 pad 8: matrix.sel_kfp.k_daq_2-coil_n -> coil_n-14
- K15 pad 7: matrix.sel_kfp.k_dmm_hi-coil_n -> sink_kfp_dmm_hi
- K16 pad 7: matrix.sel_kfp.k_dmm_lo-coil_n -> sink_kfp_dmm_lo
- K17 pad 7: matrix.sel_kfp.k_gnd-coil_n -> sink_kfp_gnd
- K18 pad 8: matrix.sel_kfp.k_logic_1-coil_n -> coil_n-16
- K19 pad 8: matrix.sel_kfp.k_logic_2-coil_n -> coil_n-17
- K2 pad 8: matrix.sel_kfn.k_daq_1-coil_n -> coil_n-18
- K20 pad 8: matrix.sel_kfp.k_pwr-coil_n -> sink_kfp_pwr
- K21 pad 8: matrix.sel_kfp.k_scope_a-coil_n -> sink_kfp_scope_a
- K22 pad 8: matrix.sel_kfp.k_scope_b-coil_n -> sink_kfp_scope_b
- K23 pad 8: matrix.sel_ksn.k_bank-coil_n -> sink_ksn_bank
- K24 pad 8: matrix.sel_ksn.k_daq_1-coil_n -> coil_n-28
- K25 pad 8: matrix.sel_ksn.k_daq_2-coil_n -> coil_n-29
- K26 pad 7: matrix.sel_ksn.k_dmm_hi-coil_n -> sink_ksn_dmm_hi
- K27 pad 7: matrix.sel_ksn.k_dmm_lo-coil_n -> sink_ksn_dmm_lo
- K28 pad 7: matrix.sel_ksn.k_gnd-coil_n -> sink_ksn_gnd
- K29 pad 8: matrix.sel_ksn.k_logic_1-coil_n -> coil_n-30
- K3 pad 8: matrix.sel_kfn.k_daq_2-coil_n -> coil_n-20
- K30 pad 8: matrix.sel_ksn.k_logic_2-coil_n -> coil_n-31
- K31 pad 8: matrix.sel_ksn.k_pwr-coil_n -> sink_ksn_pwr
- K32 pad 8: matrix.sel_ksn.k_scope_a-coil_n -> sink_ksn_scope_a
- K33 pad 8: matrix.sel_ksn.k_scope_b-coil_n -> sink_ksn_scope_b
- K34 pad 8: matrix.sel_ksp.k_bank-coil_n -> sink_ksp_bank
- K35 pad 8: matrix.sel_ksp.k_daq_1-coil_n -> coil_n-24
- K36 pad 8: matrix.sel_ksp.k_daq_2-coil_n -> coil_n-25
- K37 pad 7: matrix.sel_ksp.k_dmm_hi-coil_n -> sink_ksp_dmm_hi
- K38 pad 7: matrix.sel_ksp.k_dmm_lo-coil_n -> sink_ksp_dmm_lo
- K39 pad 7: matrix.sel_ksp.k_gnd-coil_n -> sink_ksp_gnd
- K4 pad 7: matrix.sel_kfn.k_dmm_hi-coil_n -> sink_kfn_dmm_hi
- K40 pad 8: matrix.sel_ksp.k_logic_1-coil_n -> coil_n-26
- K41 pad 8: matrix.sel_ksp.k_logic_2-coil_n -> coil_n-27
- K42 pad 8: matrix.sel_ksp.k_pwr-coil_n -> sink_ksp_pwr
- K43 pad 8: matrix.sel_ksp.k_scope_a-coil_n -> sink_ksp_scope_a
- K44 pad 8: matrix.sel_ksp.k_scope_b-coil_n -> sink_ksp_scope_b
- K45 pad 8: matrix.sel_p1.k_bank-coil_n -> sink_p1_bank
- K46 pad 8: matrix.sel_p1.k_daq_1-coil_n -> coil_n-11
- K47 pad 8: matrix.sel_p1.k_daq_2-coil_n -> coil_n-15
- K48 pad 7: matrix.sel_p1.k_dmm_hi-coil_n -> sink_p1_dmm_hi
- K49 pad 7: matrix.sel_p1.k_dmm_lo-coil_n -> sink_p1_dmm_lo
- K5 pad 7: matrix.sel_kfn.k_dmm_lo-coil_n -> sink_kfn_dmm_lo
- K50 pad 7: matrix.sel_p1.k_gnd-coil_n -> sink_p1_gnd
- K51 pad 8: matrix.sel_p1.k_logic_1-coil_n -> coil_n-19
- K52 pad 8: matrix.sel_p1.k_logic_2-coil_n -> coil_n-23
- K53 pad 8: matrix.sel_p1.k_pwr-coil_n -> sink_p1_pwr
- K54 pad 8: matrix.sel_p1.k_scope_a-coil_n -> sink_p1_scope_a
- K55 pad 8: matrix.sel_p1.k_scope_b-coil_n -> sink_p1_scope_b
- K56 pad 8: matrix.sel_p2.k_bank-coil_n -> sink_p2_bank
- K57 pad 8: matrix.sel_p2.k_daq_1-coil_n -> coil_n
- K58 pad 8: matrix.sel_p2.k_daq_2-coil_n -> coil_n-1
- K59 pad 7: matrix.sel_p2.k_dmm_hi-coil_n -> sink_p2_dmm_hi
- K6 pad 7: matrix.sel_kfn.k_gnd-coil_n -> sink_kfn_gnd
- K60 pad 7: matrix.sel_p2.k_dmm_lo-coil_n -> sink_p2_dmm_lo
- K61 pad 7: matrix.sel_p2.k_gnd-coil_n -> sink_p2_gnd
- K62 pad 8: matrix.sel_p2.k_logic_1-coil_n -> coil_n-2
- K63 pad 8: matrix.sel_p2.k_logic_2-coil_n -> coil_n-3
- K64 pad 8: matrix.sel_p2.k_pwr-coil_n -> sink_p2_pwr
- K65 pad 8: matrix.sel_p2.k_scope_a-coil_n -> sink_p2_scope_a
- K66 pad 8: matrix.sel_p2.k_scope_b-coil_n -> sink_p2_scope_b
- K67 pad 8: matrix.sel_p3.k_bank-coil_n -> sink_p3_bank
- K68 pad 8: matrix.sel_p3.k_daq_1-coil_n -> coil_n-4
- K69 pad 8: matrix.sel_p3.k_daq_2-coil_n -> coil_n-5
- K7 pad 8: matrix.sel_kfn.k_logic_1-coil_n -> coil_n-21
- K70 pad 7: matrix.sel_p3.k_dmm_hi-coil_n -> sink_p3_dmm_hi
- K71 pad 7: matrix.sel_p3.k_dmm_lo-coil_n -> sink_p3_dmm_lo
- K72 pad 7: matrix.sel_p3.k_gnd-coil_n -> sink_p3_gnd
- K73 pad 8: matrix.sel_p3.k_logic_1-coil_n -> coil_n-6
- K74 pad 8: matrix.sel_p3.k_logic_2-coil_n -> coil_n-7
- K75 pad 8: matrix.sel_p3.k_pwr-coil_n -> sink_p3_pwr
- K76 pad 8: matrix.sel_p3.k_scope_a-coil_n -> sink_p3_scope_a
- K77 pad 8: matrix.sel_p3.k_scope_b-coil_n -> sink_p3_scope_b
- K78 pad 8: matrix.sel_p4.k_bank-coil_n -> sink_p4_bank
- K79 pad 8: matrix.sel_p4.k_daq_1-coil_n -> coil_n-8
- K8 pad 8: matrix.sel_kfn.k_logic_2-coil_n -> coil_n-22
- K80 pad 8: matrix.sel_p4.k_daq_2-coil_n -> coil_n-9
- K81 pad 7: matrix.sel_p4.k_dmm_hi-coil_n -> sink_p4_dmm_hi
- K82 pad 7: matrix.sel_p4.k_dmm_lo-coil_n -> sink_p4_dmm_lo
- K83 pad 7: matrix.sel_p4.k_gnd-coil_n -> sink_p4_gnd
- K84 pad 8: matrix.sel_p4.k_logic_1-coil_n -> coil_n-10
- K85 pad 8: matrix.sel_p4.k_logic_2-coil_n -> coil_n-12
- K86 pad 8: matrix.sel_p4.k_pwr-coil_n -> sink_p4_pwr
- K87 pad 8: matrix.sel_p4.k_scope_a-coil_n -> sink_p4_scope_a
- K88 pad 8: matrix.sel_p4.k_scope_b-coil_n -> sink_p4_scope_b
- K89 pad 7: refs.k_1k-coil_n -> sink_1k
- K9 pad 8: matrix.sel_kfn.k_pwr-coil_n -> sink_kfn_pwr
- K90 pad 7: refs.k_100k-coil_n -> sink_100k
- K91 pad 7: refs.k_short-coil_n -> sink_short
- U10 pad 14: ctl.sr9-14 -> coil_n-21
- U10 pad 15: ctl.sr9-15 -> coil_n-22
- U10 pad 16: ctl.sr9-16 -> sink_kfn_pwr
- U10 pad 17: ctl.sr9-17 -> sink_kfn_dmm_hi
- U10 pad 18: ctl-SERIN-2 -> ctl-SERIN-10
- U10 pad 3: ctl-SERIN-10 -> ctl-SERIN-9
- U10 pad 4: ctl.sr9-4 -> sink_kfn_scope_a
- U10 pad 5: ctl.sr9-5 -> sink_kfn_scope_b
- U10 pad 6: ctl.sr9-6 -> coil_n-18
- U10 pad 7: ctl.sr9-7 -> coil_n-20
- U11 pad 14: ctl.sr10-14 -> sink_ksp_scope_b
- U11 pad 15: ctl.sr10-15 -> coil_n-24
- U11 pad 16: ctl.sr10-16 -> coil_n-25
- U11 pad 17: ctl.sr10-17 -> coil_n-26
- U11 pad 18: ctl-SERIN-1 -> ctl-SERIN-2
- U11 pad 3: ctl-SERIN-2 -> ctl-SERIN-10
- U11 pad 4: ctl.sr10-4 -> sink_kfn_dmm_lo
- U11 pad 5: ctl.sr10-5 -> sink_kfn_gnd
- U11 pad 6: ctl.sr10-6 -> sink_ksp_bank
- U11 pad 7: ctl.sr10-7 -> sink_ksp_scope_a
- U12 pad 14: ctl.sr11-14 -> sink_ksp_gnd
- U12 pad 15: ctl.sr11-15 -> sink_ksn_bank
- U12 pad 16: ctl.sr11-16 -> sink_ksn_scope_a
- U12 pad 17: ctl.sr11-17 -> sink_ksn_scope_b
- U12 pad 18: ctl-SERIN-3 -> ctl-SERIN-1
- U12 pad 3: ctl-SERIN-1 -> ctl-SERIN-2
- U12 pad 4: ctl.sr11-4 -> coil_n-27
- U12 pad 5: ctl.sr11-5 -> sink_ksp_pwr
- U12 pad 6: ctl.sr11-6 -> sink_ksp_dmm_hi
- U12 pad 7: ctl.sr11-7 -> sink_ksp_dmm_lo
- U13 pad 14: ctl.sr12-14 -> sink_ksn_pwr
- U13 pad 15: ctl.sr12-15 -> sink_ksn_dmm_hi
- U13 pad 16: ctl.sr12-16 -> sink_ksn_dmm_lo
- U13 pad 17: ctl.sr12-17 -> sink_ksn_gnd
- U13 pad 18: SEROUT -> ctl-SERIN-3
- U13 pad 3: ctl-SERIN-3 -> ctl-SERIN-1
- U13 pad 4: ctl.sr12-4 -> coil_n-28
- U13 pad 5: ctl.sr12-5 -> coil_n-29
- U13 pad 6: ctl.sr12-6 -> coil_n-30
- U13 pad 7: ctl.sr12-7 -> coil_n-31
- U14 pad 1: nG -> (no net)
- U14 pad 2: lv -> hv
- U14 pad 3: hv -> ctl-SERIN-3
- U14 pad 4: WDI -> sink_1k
- U14 pad 5: hv -> sink_100k
- U15 pad 1: EN -> nG
- U15 pad 2: PG -> lv
- U15 pad 3: FB -> hv
- U15 pad 4: hv -> WDI
- U15 pad 5: lv -> hv
- U16 pad 1: c_boot-power-hv -> EN
- U16 pad 2: C -> PG
- U16 pad 3: C -> FB
- U16 pad 4: SS -> hv
- U16 pad 5: VSENSE -> lv
- U16 pad 6: COMP -> SW
- U16 pad 7: lv -> EN
- U17 pad 1: EN -> c_boot-power-hv
- U17 pad 2: sel_p4-coil_bus-hv -> C
- U17 pad 3: lv -> C
- U17 pad 4: hv -> SS
- U17 pad 5: power-scl -> VSENSE
- U17 pad 6: power-sda -> COMP
- U17 pad 8: lv -> power-lv
- U18 pad 1: v3v3-hv -> EN
- U18 pad 2: power-FB -> sel_p4-coil_bus-hv
- U18 pad 3: (no net) -> lv
- U18 pad 4: lv -> hv
- U18 pad 5: EN -> power-scl
- U18 pad 6: c_nr-power-hv -> power-sda
- U18 pad 7: DNC -> lv
- U18 pad 8: EN -> lv
- U19 pad 1: IN_Apos -> v3v3-hv
- U19 pad 2: IN_Aneg -> power-FB
- U19 pad 3: IN_Bpos -> (no net)
- U19 pad 4: IN_Apos -> lv
- U19 pad 5: lv -> EN
- U19 pad 6: vcheck_lo -> c_nr-power-hv
- U19 pad 7: vcheck_hi -> DNC
- U19 pad 8: v3v3-hv -> EN
- U2 pad 1: (no net) -> 1
- U2 pad 10: lv -> scl
- U2 pad 11: lv -> WDI
- U2 pad 12: RCK -> 12
- U2 pad 13: SRCK -> 13
- U2 pad 18: ctl-SERIN -> 18
- U2 pad 19: lv -> 19
- U2 pad 2: hv -> 2
- U2 pad 20: (no net) -> 20
- U2 pad 3: SERIN -> 3
- U2 pad 4: 4 -> SRCK
- U2 pad 5: 5 -> SERIN
- U2 pad 6: 6 -> RCK
- U2 pad 7: 7 -> nG
- U2 pad 8: hv -> 8
- U2 pad 9: nG -> sda
- U20 pad 1: prot_kfp-IN_Apos -> IN_Apos
- U20 pad 2: prot_kfp.comp-IN_Aneg -> IN_Aneg
- U20 pad 3: prot_kfp.comp-IN_Bpos -> IN_Bpos
- U20 pad 4: prot_kfp-IN_Apos -> IN_Apos
- U20 pad 6: prot_kfp-vcheck_lo -> vcheck_lo
- U20 pad 7: prot_kfp-vcheck_hi -> vcheck_hi
- U21 pad 1: prot_ksn-IN_Apos -> tip-5
- U21 pad 2: prot_ksn.comp-IN_Aneg -> node
- U22 pad 1: prot_ksp-IN_Apos -> prot_kfp-IN_Apos
- U22 pad 2: prot_ksp.comp-IN_Aneg -> prot_kfp.comp-IN_Aneg
- U22 pad 3: prot_ksp.comp-IN_Bpos -> prot_kfp.comp-IN_Bpos
- U22 pad 4: prot_ksp-IN_Apos -> prot_kfp-IN_Apos
- U22 pad 6: prot_ksp-vcheck_lo -> prot_kfp-vcheck_lo
- U22 pad 7: prot_ksp-vcheck_hi -> prot_kfp-vcheck_hi
- U23 pad 1: prot_p1-IN_Apos -> tip-4
- U23 pad 2: prot_p1.comp-IN_Aneg -> node-1
- U24 pad 1: prot_p2-IN_Apos -> prot_ksn-IN_Apos
- U24 pad 2: prot_p2.comp-IN_Aneg -> prot_ksn.comp-IN_Aneg
- U24 pad 3: prot_p2.comp-IN_Bpos -> prot_ksn.comp-IN_Bpos
- U24 pad 4: prot_p2-IN_Apos -> prot_ksn-IN_Apos
- U24 pad 6: prot_p2-vcheck_lo -> prot_ksn-vcheck_lo
- U24 pad 7: prot_p2-vcheck_hi -> prot_ksn-vcheck_hi
- U25 pad 1: prot_p3-IN_Apos -> tip-7
- U25 pad 2: prot_p3.comp-IN_Aneg -> node-2
- U26 pad 1: prot_p4-IN_Apos -> prot_ksp-IN_Apos
- U26 pad 2: prot_p4.comp-IN_Aneg -> prot_ksp.comp-IN_Aneg
- U26 pad 3: prot_p4.comp-IN_Bpos -> prot_ksp.comp-IN_Bpos
- U26 pad 4: prot_p4-IN_Apos -> prot_ksp-IN_Apos
- U26 pad 6: prot_p4-vcheck_lo -> prot_ksp-vcheck_lo
- U26 pad 7: prot_p4-vcheck_hi -> prot_ksp-vcheck_hi
- U27 pad 1: tip-5 -> tip-6
- U27 pad 2: node -> node-3
- U28 pad 1: tip-4 -> prot_p1-IN_Apos
- U28 pad 2: node-1 -> prot_p1.comp-IN_Aneg
- U29 pad 1: tip-7 -> tip
- U29 pad 2: node-2 -> node-4
- U3 pad 14: ctl.sr2-14 -> coil_n-15
- U3 pad 15: ctl.sr2-15 -> coil_n-19
- U3 pad 16: ctl.sr2-16 -> coil_n-23
- U3 pad 17: ctl.sr2-17 -> sink_p1_pwr
- U3 pad 18: ctl-SERIN-4 -> ctl-SERIN
- U3 pad 3: ctl-SERIN -> SERIN
- U3 pad 4: ctl.sr2-4 -> sink_p1_bank
- U3 pad 5: ctl.sr2-5 -> sink_p1_scope_a
- U3 pad 6: ctl.sr2-6 -> sink_p1_scope_b
- U3 pad 7: ctl.sr2-7 -> coil_n-11
- U30 pad 1: tip-6 -> prot_p2-IN_Apos
- U30 pad 2: node-3 -> prot_p2.comp-IN_Aneg
- U31 pad 1: tip -> tip-1
- U31 pad 2: node-4 -> node-5
- U32 pad 1: tip-1 -> prot_p3-IN_Apos
- U32 pad 2: node-5 -> prot_p3.comp-IN_Aneg
- U34 pad 1: tip-3 -> prot_p4-IN_Apos
- U34 pad 2: node-7 -> prot_p4.comp-IN_Aneg
- U4 pad 14: ctl.sr3-14 -> sink_p2_scope_a
- U4 pad 15: ctl.sr3-15 -> sink_p2_scope_b
- U4 pad 16: ctl.sr3-16 -> coil_n
- U4 pad 17: ctl.sr3-17 -> coil_n-1
- U4 pad 18: ctl-SERIN-5 -> ctl-SERIN-4
- U4 pad 3: ctl-SERIN-4 -> ctl-SERIN
- U4 pad 4: ctl.sr3-4 -> sink_p1_dmm_hi
- U4 pad 5: ctl.sr3-5 -> sink_p1_dmm_lo
- U4 pad 6: ctl.sr3-6 -> sink_p1_gnd
- U4 pad 7: ctl.sr3-7 -> sink_p2_bank
- U5 pad 14: ctl.sr4-14 -> sink_p2_dmm_lo
- U5 pad 15: ctl.sr4-15 -> sink_p2_gnd
- U5 pad 16: ctl.sr4-16 -> sink_p3_bank
- U5 pad 17: ctl.sr4-17 -> sink_p3_scope_a
- U5 pad 18: ctl-SERIN-6 -> ctl-SERIN-5
- U5 pad 3: ctl-SERIN-5 -> ctl-SERIN-4
- U5 pad 4: ctl.sr4-4 -> coil_n-2
- U5 pad 5: ctl.sr4-5 -> coil_n-3
- U5 pad 6: ctl.sr4-6 -> sink_p2_pwr
- U5 pad 7: ctl.sr4-7 -> sink_p2_dmm_hi
- U6 pad 14: ctl.sr5-14 -> coil_n-7
- U6 pad 15: ctl.sr5-15 -> sink_p3_pwr
- U6 pad 16: ctl.sr5-16 -> sink_p3_dmm_hi
- U6 pad 17: ctl.sr5-17 -> sink_p3_dmm_lo
- U6 pad 18: ctl-SERIN-7 -> ctl-SERIN-6
- U6 pad 3: ctl-SERIN-6 -> ctl-SERIN-5
- U6 pad 4: ctl.sr5-4 -> sink_p3_scope_b
- U6 pad 5: ctl.sr5-5 -> coil_n-4
- U6 pad 6: ctl.sr5-6 -> coil_n-5
- U6 pad 7: ctl.sr5-7 -> coil_n-6
- U7 pad 14: ctl.sr6-14 -> coil_n-8
- U7 pad 15: ctl.sr6-15 -> coil_n-9
- U7 pad 16: ctl.sr6-16 -> coil_n-10
- U7 pad 17: ctl.sr6-17 -> coil_n-12
- U7 pad 18: ctl-SERIN-8 -> ctl-SERIN-7
- U7 pad 3: ctl-SERIN-7 -> ctl-SERIN-6
- U7 pad 4: ctl.sr6-4 -> sink_p3_gnd
- U7 pad 5: ctl.sr6-5 -> sink_p4_bank
- U7 pad 6: ctl.sr6-6 -> sink_p4_scope_a
- U7 pad 7: ctl.sr6-7 -> sink_p4_scope_b
- U8 pad 14: ctl.sr7-14 -> sink_kfp_bank
- U8 pad 15: ctl.sr7-15 -> sink_kfp_scope_a
- U8 pad 16: ctl.sr7-16 -> sink_kfp_scope_b
- U8 pad 17: ctl.sr7-17 -> coil_n-13
- U8 pad 18: ctl-SERIN-9 -> ctl-SERIN-8
- U8 pad 3: ctl-SERIN-8 -> ctl-SERIN-7
- U8 pad 4: ctl.sr7-4 -> sink_p4_pwr
- U8 pad 5: ctl.sr7-5 -> sink_p4_dmm_hi
- U8 pad 6: ctl.sr7-6 -> sink_p4_dmm_lo
- U8 pad 7: ctl.sr7-7 -> sink_p4_gnd
- U9 pad 14: ctl.sr8-14 -> sink_kfp_dmm_hi
- U9 pad 15: ctl.sr8-15 -> sink_kfp_dmm_lo
- U9 pad 16: ctl.sr8-16 -> sink_kfp_gnd
- U9 pad 17: ctl.sr8-17 -> sink_kfn_bank
- U9 pad 18: ctl-SERIN-10 -> ctl-SERIN-9
- U9 pad 3: ctl-SERIN-9 -> ctl-SERIN-8
- U9 pad 4: ctl.sr8-4 -> coil_n-14
- U9 pad 5: ctl.sr8-5 -> coil_n-16
- U9 pad 6: ctl.sr8-6 -> coil_n-17
- U9 pad 7: ctl.sr8-7 -> sink_kfp_pwr

Commit message: Placement engine v3 + quality gates: kill the routing trial-and-error
Root cause of router struggles was connectivity-blind placement with
hardcoded pitches. Rebuilt as code we own and iterate:

- scripts/placement_score.py: pre-route GATE (courtyard overlaps,
  off-board) + HPWL score. Placements that fail never reach the router.
- Channel map v2 (LOCALITY): TPIC 1-8 each sink their own relay tree's
  8 G6K coils and sit directly above that tree; TPIC 9-11 sink the reed
  bank; TPIC 12 the reference block. 91 coil nets become short locals
  instead of cross-board runs. coil-channel-map.md updated (firmware
  shares the table).
- place_and_zone.py v3: pitches DERIVED from measured courtyards;
  relays grouped per tree by net classification (instance-path nets,
  sink aliases, drain-number decode -- the shared rail being named
  'sel_p4-coil_bus-hv' poisoned naive matching); TPICs placed by
  net-sharing vote with their relays; board grown to 200x175 from the
  measured vertical budget.
- Result: GATE PASS (was 12+ overlaps), HPWL 18862mm vs 20587 baseline.

freerouting stays the stock released jar (GPL source available, but the
placement was the lever, not the router).

Co-Authored-By: Claude Fable 5 <noreply@anthropic.com>
Connections:
- K13 pad 8: coil_n-13 -> coil_n-12
- K14 pad 8: coil_n-14 -> coil_n-13
- K18 pad 8: coil_n-16 -> coil_n-14
- K19 pad 8: coil_n-17 -> coil_n-15
- K2 pad 8: coil_n-18 -> coil_n-17
- K24 pad 8: coil_n-28 -> coil_n-27
- K25 pad 8: coil_n-29 -> coil_n-28
- K29 pad 8: coil_n-30 -> coil_n-29
- K3 pad 8: coil_n-20 -> coil_n-18
- K30 pad 8: coil_n-31 -> coil_n-30
- K35 pad 8: coil_n-24 -> coil_n-22
- K36 pad 8: coil_n-25 -> coil_n-23
- K40 pad 8: coil_n-26 -> coil_n-24
- K41 pad 8: coil_n-27 -> coil_n-25
- K46 pad 8: coil_n-11 -> coil_n-16
- K47 pad 8: coil_n-15 -> coil_n-21
- K51 pad 8: coil_n-19 -> coil_n-26
- K52 pad 8: coil_n-23 -> coil_n-31
- K7 pad 8: coil_n-21 -> coil_n-19
- K8 pad 8: coil_n-22 -> coil_n-20
- K85 pad 8: coil_n-12 -> coil_n-11
- U10 pad 14: coil_n-21 -> coil_n-28
- U10 pad 15: coil_n-22 -> coil_n-29
- U10 pad 16: sink_kfn_pwr -> coil_n-30
- U10 pad 17: sink_kfn_dmm_hi -> sink_ksn_pwr
- U10 pad 4: sink_kfn_scope_a -> sink_ksn_bank
- U10 pad 5: sink_kfn_scope_b -> sink_ksn_scope_a
- U10 pad 6: coil_n-18 -> sink_ksn_scope_b
- U10 pad 7: coil_n-20 -> coil_n-27
- U11 pad 14: sink_ksp_scope_b -> sink_p2_dmm_lo
- U11 pad 15: coil_n-24 -> sink_p2_gnd
- U11 pad 16: coil_n-25 -> sink_p3_dmm_hi
- U11 pad 17: coil_n-26 -> sink_p3_dmm_lo
- U11 pad 4: sink_kfn_dmm_lo -> sink_p1_dmm_hi
- U11 pad 5: sink_kfn_gnd -> sink_p1_dmm_lo
- U11 pad 6: sink_ksp_bank -> sink_p1_gnd
- U11 pad 7: sink_ksp_scope_a -> sink_p2_dmm_hi
- U12 pad 14: sink_ksp_gnd -> sink_kfp_dmm_hi
- U12 pad 15: sink_ksn_bank -> sink_kfp_dmm_lo
- U12 pad 16: sink_ksn_scope_a -> sink_kfp_gnd
- U12 pad 17: sink_ksn_scope_b -> sink_kfn_dmm_hi
- U12 pad 4: coil_n-27 -> sink_p3_gnd
- U12 pad 5: sink_ksp_pwr -> sink_p4_dmm_hi
- U12 pad 6: sink_ksp_dmm_hi -> sink_p4_dmm_lo
- U12 pad 7: sink_ksp_dmm_lo -> sink_p4_gnd
- U13 pad 14: sink_ksn_pwr -> sink_ksp_gnd
- U13 pad 4: coil_n-28 -> sink_kfn_dmm_lo
- U13 pad 5: coil_n-29 -> sink_kfn_gnd
- U13 pad 6: coil_n-30 -> sink_ksp_dmm_hi
- U13 pad 7: coil_n-31 -> sink_ksp_dmm_lo
- U3 pad 14: coil_n-15 -> coil_n-21
- U3 pad 15: coil_n-19 -> coil_n-26
- U3 pad 16: coil_n-23 -> coil_n-31
- U3 pad 7: coil_n-11 -> coil_n-16
- U4 pad 14: sink_p2_scope_a -> coil_n-1
- U4 pad 15: sink_p2_scope_b -> coil_n-2
- U4 pad 16: coil_n -> coil_n-3
- U4 pad 17: coil_n-1 -> sink_p2_pwr
- U4 pad 4: sink_p1_dmm_hi -> sink_p2_bank
- U4 pad 5: sink_p1_dmm_lo -> sink_p2_scope_a
- U4 pad 6: sink_p1_gnd -> sink_p2_scope_b
- U4 pad 7: sink_p2_bank -> coil_n
- U5 pad 14: sink_p2_dmm_lo -> coil_n-5
- U5 pad 15: sink_p2_gnd -> coil_n-6
- U5 pad 16: sink_p3_bank -> coil_n-7
- U5 pad 17: sink_p3_scope_a -> sink_p3_pwr
- U5 pad 4: coil_n-2 -> sink_p3_bank
- U5 pad 5: coil_n-3 -> sink_p3_scope_a
- U5 pad 6: sink_p2_pwr -> sink_p3_scope_b
- U5 pad 7: sink_p2_dmm_hi -> coil_n-4
- U6 pad 14: coil_n-7 -> coil_n-9
- U6 pad 15: sink_p3_pwr -> coil_n-10
- U6 pad 16: sink_p3_dmm_hi -> coil_n-11
- U6 pad 17: sink_p3_dmm_lo -> sink_p4_pwr
- U6 pad 4: sink_p3_scope_b -> sink_p4_bank
- U6 pad 5: coil_n-4 -> sink_p4_scope_a
- U6 pad 6: coil_n-5 -> sink_p4_scope_b
- U6 pad 7: coil_n-6 -> coil_n-8
- U7 pad 14: coil_n-8 -> coil_n-13
- U7 pad 15: coil_n-9 -> coil_n-14
- U7 pad 16: coil_n-10 -> coil_n-15
- U7 pad 17: coil_n-12 -> sink_kfp_pwr
- U7 pad 4: sink_p3_gnd -> sink_kfp_bank
- U7 pad 5: sink_p4_bank -> sink_kfp_scope_a
- U7 pad 6: sink_p4_scope_a -> sink_kfp_scope_b
- U7 pad 7: sink_p4_scope_b -> coil_n-12
- U8 pad 14: sink_kfp_bank -> coil_n-18
- U8 pad 15: sink_kfp_scope_a -> coil_n-19
- U8 pad 16: sink_kfp_scope_b -> coil_n-20
- U8 pad 17: coil_n-13 -> sink_kfn_pwr
- U8 pad 4: sink_p4_pwr -> sink_kfn_bank
- U8 pad 5: sink_p4_dmm_hi -> sink_kfn_scope_a
- U8 pad 6: sink_p4_dmm_lo -> sink_kfn_scope_b
- U8 pad 7: sink_p4_gnd -> coil_n-17
- U9 pad 14: sink_kfp_dmm_hi -> coil_n-23
- U9 pad 15: sink_kfp_dmm_lo -> coil_n-24
- U9 pad 16: sink_kfp_gnd -> coil_n-25
- U9 pad 17: sink_kfn_bank -> sink_ksp_pwr
- U9 pad 4: coil_n-14 -> sink_ksp_bank
- U9 pad 5: coil_n-16 -> sink_ksp_scope_a
- U9 pad 6: coil_n-17 -> sink_ksp_scope_b
- U9 pad 7: sink_kfp_pwr -> coil_n-22
